Commit message: rtabmap support

File: quadruped_gazebo/urdf/a1/a1_rs.xacro (robot description, xacro)
@@ -43,10 +43,7 @@
     <child link="trunk"/>
   </joint>
-  <xacro:depth_sensor>
+  <xacro:depth_sensor camera_link="camera_link_1" camera_name="camera_1">
       <origin xyz="0.3 0 0.05" rpy="0 0 0"/>
   </xacro:depth_sensor>
-  <!-- <xacro:sensor_d435 parent="base" use_nominal_extrinsics="false" use_mesh="true">
-    <origin xyz="0.5 0 0.1" rpy="0 0 0"/>
-  </xacro:sensor_d435> -->
   <link name="trunk">
     <visual>

File: quadruped_gazebo/urdf/depth_sensor.urdf.xacro (robot description, xacro)
@@ -1,6 +1,6 @@
 <robot xmlns:xacro="http://ros.org/wiki/xacro">
   <xacro:property name="M_PI" value="3.1415926535897931" />
-  <xacro:macro name="depth_sensor" params="*origin">
-    <link name="camera_link">
+  <xacro:macro name="depth_sensor" params="*origin camera_link:=camera_link camera_name:=camera">
+    <link name="${camera_link}">
       <visual>
         <origin xyz="0 0 0" rpy="0 0 0"/>
@@ -27,5 +27,5 @@
       </inertial>
     </link>
-    <gazebo reference="camera_link">
+    <gazebo reference="${camera_link}">
       <visual>
         <material>
@@ -39,5 +39,5 @@
     <joint name="camera_to_base_link" type="fixed">
       <parent link="base_link"/>
-      <child link="camera_link"/>
+      <child link="${camera_link}"/>
       <xacro:insert_block name="origin" />
     </joint>
@@ -45,9 +45,9 @@
     <joint name="camera_depth_joint" type="fixed">
       <origin xyz="0 0 0" rpy="-1.57 0 -1.57"/>
-      <parent link="camera_link"/>
+      <parent link="${camera_link}"/>
       <child link="camera_depth_link"/>
     </joint>
     <!-- https://github.com/ros-simulation/gazebo_ros_pkgs/wiki/ROS-2-Migration:-Camera#gazebo_ros_camera -->
-    <gazebo reference="camera_link">
+    <gazebo reference="${camera_link}">
       <sensor name="camera" type="depth">
         <always_on>true</always_on>
@@ -63,7 +63,9 @@
         <plugin name="camera_controller" filename="libgazebo_ros_camera.so">
           <ros>
-            <remapping>/camera/camera_info:=/camera/camera_info</remapping>
-            <remapping>/camera/image_raw:=/camera/image_raw</remapping>
-            <remapping>/camera/points:=/camera/depth/color/points</remapping>
+            <remapping>/camera/camera_info:=${camera_name}/camera/camera_info</remapping>
+            <remapping>/camera/image_raw:=${camera_name}/camera/image_raw</remapping>
+            <remapping>/camera/points:=${camera_name}/camera/depth/color/points</remapping>
+            <remapping>/camera/depth/camera_info:=${camera_name}/camera/depth/camera_info</remapping>
+            <remapping>/camera/depth/image_raw:=${camera_name}/camera/depth/image_raw</remapping>
             <!-- <remapping>/camera/depth/image_raw:=/camera/depth/image_rect_raw</remapping> -->
           </ros>

Commit message: dual cam

File: quadruped_gazebo/urdf/a1/a1_rs.xacro (robot description, xacro)
@@ -45,4 +45,7 @@
   <xacro:depth_sensor camera_link="camera_link_1" camera_name="camera_1">
       <origin xyz="0.3 0 0.05" rpy="0 0 0"/>
+  </xacro:depth_sensor>
+  <xacro:depth_sensor camera_link="camera_link_2" camera_name="camera_2">
+      <origin xyz="-0.3 0 0.05" rpy="0 0 3.14159"/>
   </xacro:depth_sensor>
   <link name="trunk">

File: quadruped_gazebo/urdf/depth_sensor.urdf.xacro (robot description, xacro)
@@ -37,21 +37,21 @@
       </visual>
     </gazebo>rgb(213,28,40)
-    <joint name="camera_to_base_link" type="fixed">
+    <joint name="${camera_name}_to_base_link" type="fixed">
       <parent link="base_link"/>
       <child link="${camera_link}"/>
       <xacro:insert_block name="origin" />
     </joint>
-    <link name="camera_depth_link"/>
-    <joint name="camera_depth_joint" type="fixed">
+    <link name="${camera_name}_depth_link"/>
+    <joint name="${camera_name}_depth_joint" type="fixed">
       <origin xyz="0 0 0" rpy="-1.57 0 -1.57"/>
       <parent link="${camera_link}"/>
-      <child link="camera_depth_link"/>
+      <child link="${camera_name}_depth_link"/>
     </joint>
     <!-- https://github.com/ros-simulation/gazebo_ros_pkgs/wiki/ROS-2-Migration:-Camera#gazebo_ros_camera -->
     <gazebo reference="${camera_link}">
-      <sensor name="camera" type="depth">
+      <sensor name="${camera_name}" type="depth">
         <always_on>true</always_on>
         <update_rate>30.0</update_rate>
-        <camera name="camera">
+        <camera name="${camera_name}">
           <horizontal_fov>1.50098</horizontal_fov>
           <image>
@@ -63,9 +63,9 @@
         <plugin name="camera_controller" filename="libgazebo_ros_camera.so">
           <ros>
-            <remapping>/camera/camera_info:=${camera_name}/camera/camera_info</remapping>
-            <remapping>/camera/image_raw:=${camera_name}/camera/image_raw</remapping>
-            <remapping>/camera/points:=${camera_name}/camera/depth/color/points</remapping>
-            <remapping>/camera/depth/camera_info:=${camera_name}/camera/depth/camera_info</remapping>
-            <remapping>/camera/depth/image_raw:=${camera_name}/camera/depth/image_raw</remapping>
+            <remapping>/${camera_name}/camera_info:=${camera_name}/camera_info</remapping>
+            <remapping>/${camera_name}/image_raw:=${camera_name}/image_raw</remapping>
+            <remapping>/${camera_name}/points:=${camera_name}/depth/color/points</remapping>
+            <remapping>/${camera_name}/depth/camera_info:=${camera_name}/depth/camera_info</remapping>
+            <remapping>/${camera_name}/depth/image_raw:=${camera_name}/depth/image_raw</remapping>
             <!-- <remapping>/camera/depth/image_raw:=/camera/depth/image_rect_raw</remapping> -->
           </ros>
@@ -73,5 +73,5 @@
           <max_depth>3.0</max_depth>
           <hack_baseline>0.07</hack_baseline>
-          <frame_name>camera_depth_link</frame_name>
+          <frame_name>${camera_name}_depth_link</frame_name>
           <distortion_k1>0.00000001</distortion_k1>
           <distortion_k2>0.00000001</distortion_k2>
